File: KiCAD/ChuaCircuit/ChuaCircuit.kicad_pcb (KiCad board)
At the start: 2 copper layers, 30 x 50 mm, 23 parts, among them X1 TP3, Y1 TP2

Commit message: Updated PCB according to new changes
Parts:
- added C10: 0.1u, Capacitor_SMD:C_0603_1608Metric, F.Cu at (138.0, 89.8)
- added C11: 0.01u, Capacitor_SMD:C_0603_1608Metric, F.Cu at (141.0, 89.8)
- added C4: .01u, Capacitor_SMD:C_0603_1608Metric, F.Cu at (133.5, 86.3)
- added C5: 0.1u, Capacitor_SMD:C_0603_1608Metric, F.Cu at (136.5, 86.3)
- added C6: 0.1u, Capacitor_SMD:C_0603_1608Metric, F.Cu at (139.5, 86.3)
- added C7: 0.01u, Capacitor_SMD:C_0603_1608Metric, F.Cu at (142.5, 86.3)
- added C8: 0.1u, Capacitor_SMD:C_0603_1608Metric, F.Cu at (144.0, 89.8)
- added C9: 0.01u, Capacitor_SMD:C_0603_1608Metric, F.Cu at (135.0, 89.8)
- +VCC: renamed from VIN1; value Male_Header_1x1 -> J1
- -VCC: renamed from GND1; value Male_Header_1x1 -> J1
- moved C3 28.6 mm to (146.5, 94.5), turned to 90 degrees
- moved R3 27.2 mm to (146.5, 98.8), turned to 90 degrees
- moved R6 21.9 mm to (146.5, 102.5), turned to 90 degrees
- moved R1 21.5 mm to (130.5, 94.8), turned to -90 degrees
- moved R2 21.5 mm to (130.5, 98.3), turned to -90 degrees
- moved C1 14.6 mm to (134.7, 115.0)
- moved R4 13.1 mm to (130.5, 106.0), turned to -90 degrees
- moved R5 13.0 mm to (130.5, 109.7), turned to -90 degrees
- moved R7 10.5 mm to (146.5, 105.8), turned to 90 degrees
- moved R8 10.5 mm to (146.5, 109.3), turned to 90 degrees
- moved C2 9.66 mm to (140.5, 115.5)
- moved R9 9.57 mm to (145.2, 113.5)
- moved RV2 6.58 mm to (150.5, 112.5)
- moved CHUA_OUT 5.02 mm to (126.5, 77.0)
- moved GND 5.02 mm to (126.5, 87.0)
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- renumbered OUTPUT1 to CHUA_OUT, GND2 to GND
Connections:
- -VCC pad 1: GND -> Net-(-VCC1-Pin_1)
- OPA1 pad 11: GND -> Net-(-VCC1-Pin_1)
- OPA2 pad 4: GND -> Net-(OPA2C-V-)
Routing:
- net GND: track 102.8 -> 0.00 mm
- net VCC: track 33.6 -> 59.9 mm
- net Net-(-VCC1-Pin_1): track 0.00 -> 19.3 mm
- net Net-(OPA2C-V-): track 0.00 -> 17.3 mm, vias 0 -> 1
- net Net-(OPA1-Pad1): track 26.3 -> 9.24 mm
- net Net-(OPA1-Pad14): track 53.8 -> 41.3 mm
- net Net-(OPA1A--): track 27.5 -> 17.4 mm, vias 0 -> 1
- net Net-(OPA1C--): track 28.0 -> 20.0 mm, vias 0 -> 1
- net Net-(OPA1-Pad7): track 11.4 -> 8.53 mm
- net Net-(OPA1B--): track 19.0 -> 21.3 mm, vias 0 -> 1
- net Net-(C3-Pad1): track 20.6 -> 22.6 mm
- net Net-(OPA1C-+): track 48.7 -> 47.1 mm, vias 0 -> 1
- net Net-(OPA1D-+): track 28.0 -> 26.6 mm, vias 0 -> 1
- net Net-(OPA1A-+): track 80.4 -> 79.1 mm
Other:
- board size 30 x 50 mm -> 29.5 x 47 mm
- board text added: "Chua Circuit V1.0"
- board text added: "Justin Nguyen's"
- board text removed: "Justin Nguyen's Chua Circuit V1.0"

Commit message: Changed op-amp IC footprint to SMT style
Parts:
- OPA1: footprint SamacSys_Parts:TL084 -> SamacSys_Parts:SOIC127P600X175-14N
- OPA2: footprint SamacSys_Parts:TL082 -> SamacSys_Parts:SOIC127P600X175-8N
- moved CHUA_OUT1 28.6 mm to (150.5, 92.5)
- moved +VCC1 28.3 mm to (126.5, 92.5)
- moved C3 21.0 mm to (146.5, 115.5)
- moved -VCC1 20.1 mm to (131.0, 92.5)
- moved GND2 15.0 mm to (126.5, 102.0)
- moved OPA2 13.8 mm to (138.0, 93.0)
- moved C10 11.7 mm to (138.0, 101.5)
- moved C11 11.7 mm to (141.0, 101.5)
- moved C9 11.7 mm to (135.0, 101.5)
- moved C4 11.7 mm to (131.0, 97.7)
- moved C5 11.7 mm to (134.0, 97.7)
- moved C6 11.7 mm to (137.0, 97.7)
- moved C7 11.7 mm to (140.0, 97.7)
- moved X1 10.0 mm to (126.5, 107.0)
- moved C8 8.01 mm to (143.0, 97.7)
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- renumbered +VCC to +VCC1, -VCC to -VCC1, CHUA_OUT to CHUA_OUT1, GND to GND2
Routing:
- net GND: track 0.00 -> 83.2 mm, vias 0 -> 1
- net Net-(OPA1A--): track 17.4 -> 33.5 mm, vias 1 -> 2
- net VCC: track 59.9 -> 48.0 mm
- net Net-(OPA1-Pad14): track 41.3 -> 31.5 mm, vias 2 -> 1
- net Net-(C3-Pad1): track 22.6 -> 14.7 mm
- net Net-(CHUA_OUT1-Pin_1): track 11.0 -> 18.8 mm, vias 0 -> 1
- net Net-(OPA1C-+): track 47.1 -> 40.7 mm, vias 1 -> 2
- net Net-(OPA1C--): track 20.0 -> 14.7 mm, vias 1 -> 0
- net Net-(OPA2C-V-): track 17.3 -> 12.5 mm, vias 1 -> 0
- net Net-(OPA1A-+): track 79.1 -> 74.8 mm, vias 0 -> 1
- net Net-(-VCC1-Pin_1): track 19.3 -> 17.1 mm
- net Net-(OPA1-Pad1): track 9.24 -> 7.19 mm
- net Net-(OPA1D-+): track 26.6 -> 24.9 mm
- net Net-(OPA1B--): track 21.3 -> 20.1 mm, vias 1 -> 2
- net Net-(OPA1-Pad7): track 8.53 -> 7.89 mm
Other:
- board size 29.5 x 47 mm -> 29.5 x 31 mm
