File: KiCAD/ChuaCircuit/ChuaCircuit.kicad_sch (KiCad schematic)
At the start: 31 parts, among them X1 TP3, Y1 TP2

Commit message: Fixed errors with schematic
Parts:
- C10, C11, C4, C5, C6, C7, C8, C9: footprint (none) -> Capacitor_SMD:C_0603_1608Metric
- renumbered +VCC to +VCC1, -VCC to -VCC1, CHUA_OUT to CHUA_OUT1
Changed lines of the file:
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@@
 			)
 		)
-		(property "Footprint" ""
+		(property "Footprint" "Capacitor_SMD:C_0603_1608Metric"
 			(at 162.2552 161.29 0)
 			(effects
@@
 			)
 		)
-		(property "Footprint" ""
+		(property "Footprint" "Capacitor_SMD:C_0603_1608Metric"
 			(at 126.6952 161.29 0)
 			(effects
@@
 		(on_board yes)
 		(dnp no)
-		(property "Reference" "-VCC"
+		(property "Reference" "-VCC1"
 			(at 77.47 130.048 90)
 			(effects
@@
 			(project "ChuaCircuit"
 				(path "/076f7681-7b7c-4ede-84a6-3e9abd09d9f7"
-					(reference "-VCC")
+					(reference "-VCC1")
 					(unit 1)
 				)
@@
 		(on_board yes)
 		(dnp no)
-		(property "Reference" "+VCC"
+		(property "Reference" "+VCC1"
 			(at 56.388 130.556 90)
 			(effects
@@
 			(project ""
 				(path "/076f7681-7b7c-4ede-84a6-3e9abd09d9f7"
-					(reference "+VCC")
+					(reference "+VCC1")
 					(unit 1)
 				)
@@
 			)
 		)
-		(property "Footprint" ""
+		(property "Footprint" "Capacitor_SMD:C_0603_1608Metric"
 			(at 169.8752 161.29 0)
 			(effects
@@
 			)
 		)
-		(property "Footprint" ""
+		(property "Footprint" "Capacitor_SMD:C_0603_1608Metric"
 			(at 79.7052 161.29 0)
 			(effects
@@
 			)
 		)
-		(property "Footprint" ""
+		(property "Footprint" "Capacitor_SMD:C_0603_1608Metric"
 			(at 87.3252 161.29 0)
 			(effects
@@
 			)
 		)
-		(property "Footprint" ""
+		(property "Footprint" "Capacitor_SMD:C_0603_1608Metric"
 			(at 46.6852 161.29 0)
 			(effects
@@
 		(on_board yes)
 		(dnp no)
-		(property "Reference" "CHUA_OUT"
+		(property "Reference" "CHUA_OUT1"
 			(at 179.705 29.21 0)
 			(effects
@@
 			(project ""
 				(path "/076f7681-7b7c-4ede-84a6-3e9abd09d9f7"
-					(reference "CHUA_OUT")
+					(reference "CHUA_OUT1")
 					(unit 1)
 				)
@@
 			)
 		)
-		(property "Footprint" ""
+		(property "Footprint" "Capacitor_SMD:C_0603_1608Metric"
 			(at 119.0752 161.29 0)
 			(effects
@@
 			)
 		)
-		(property "Footprint" ""
+		(property "Footprint" "Capacitor_SMD:C_0603_1608Metric"
 			(at 39.0652 161.29 0)
 			(effects

Commit message: Updated PCB according to new changes
Connections:
- net +VCC is gone; now on net VCC: +VCC1.1 (Pin_1), C4.1, C5.1, OPA1.4 (V+)
Changed lines of the file:
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@@
 			)
 		)
-		(property "Value" "+VCC"
+		(property "Value" "VCC"
 			(at 58.42 139.7 90)
 			(effects

Commit message: Changed op-amp IC footprint to SMT style
Parts:
- OPA1: footprint SamacSys_Parts:TL084 -> SamacSys_Parts:SOIC127P600X175-14N
- OPA2: footprint SamacSys_Parts:TL082 -> SamacSys_Parts:SOIC127P600X175-8N
Changed lines of the file:
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@@
 			)
 		)
-		(property "Footprint" "SamacSys_Parts:TL084"
+		(property "Footprint" "SamacSys_Parts:SOIC127P600X175-14N"
 			(at 185.42 86.36 0)
 			(effects
@@
 			)
 		)
-		(property "Footprint" "SamacSys_Parts:TL082"
+		(property "Footprint" "SamacSys_Parts:SOIC127P600X175-8N"
 			(at 158.75 34.29 0)
 			(effects
@@
 			)
 		)
-		(property "Footprint" "SamacSys_Parts:TL084"
+		(property "Footprint" "SamacSys_Parts:SOIC127P600X175-14N"
 			(at 83.82 78.74 0)
 			(effects
@@
 			)
 		)
-		(property "Footprint" "SamacSys_Parts:TL084"
+		(property "Footprint" "SamacSys_Parts:SOIC127P600X175-14N"
 			(at 106.68 97.79 0)
 			(effects
@@
 			)
 		)
-		(property "Footprint" "SamacSys_Parts:TL084"
+		(property "Footprint" "SamacSys_Parts:SOIC127P600X175-14N"
 			(at 166.37 91.44 0)
 			(effects
@@
 			)
 		)
-		(property "Footprint" "SamacSys_Parts:TL084"
+		(property "Footprint" "SamacSys_Parts:SOIC127P600X175-14N"
 			(at 62.23 151.13 0)
 			(effects
@@
 			)
 		)
-		(property "Footprint" "SamacSys_Parts:TL082"
+		(property "Footprint" "SamacSys_Parts:SOIC127P600X175-8N"
 			(at 144.78 149.86 0)
 			(effects
